File: Swarm_robot_project.kicad_sch (KiCad schematic)
At the start: 87 parts, among them J1 Motor_A, J2 Motor_B, J3 SW, J4 Lipo_2000mAh, J5 USB_C_Receptacle_USB2.0_16P, SW1 SW_Push, SW2 SW_Push, SW3 SW_SPDT, SW4 SW_Push, SW5 SW_POWER, U1 TPS63802DLAR, U2 MT3608, U3 BQ24075RGT, U4 DRV8833PWP, U5 STM32F103C8T6, U6 ESP32-C3-WROOM-02, U7 USBLC6-2SC6, Y1 16MHz

Commit message: UPDATE
Parts:
- R10, R11, R14, R15, R19, R20, R21, R22, R27, R28, R5: LCSC C60490 -> C25744
Changed lines of the file:
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@@
 			)
 		)
-		(property "LCSC" "C60490"
+		(property "LCSC" "C25744"
 			(at 175.26 127 0)
 			(hide yes)
@@
 			)
 		)
-		(property "LCSC" "C60490"
+		(property "LCSC" "C25744"
 			(at 260.35 167.64 0)
 			(hide yes)
@@
 			)
 		)
-		(property "LCSC" "C60490"
+		(property "LCSC" "C25744"
 			(at 66.04 128.27 0)
 			(hide yes)
@@
 			)
 		)
-		(property "LCSC" "C60490"
+		(property "LCSC" "C25744"
 			(at 82.55 52.07 0)
 			(hide yes)
@@
 			)
 		)
-		(property "LCSC" "C60490"
+		(property "LCSC" "C25744"
 			(at 260.35 118.11 0)
 			(hide yes)
@@
 			)
 		)
-		(property "LCSC" "C60490"
+		(property "LCSC" "C25744"
 			(at 63.5 118.11 0)
 			(hide yes)
@@
 			)
 		)
-		(property "LCSC" "C60490"
+		(property "LCSC" "C25744"
 			(at 81.28 57.15 0)
 			(hide yes)
@@
 			)
 		)
-		(property "LCSC" "C60490"
+		(property "LCSC" "C25744"
 			(at 379.73 105.41 0)
 			(hide yes)
@@
 			)
 		)
-		(property "LCSC" "C60490"
+		(property "LCSC" "C25744"
 			(at 177.8 58.42 0)
 			(hide yes)
@@
 			)
 		)
-		(property "LCSC" "C60490"
+		(property "LCSC" "C25744"
 			(at 177.8 127 0)
 			(hide yes)
@@
 			)
 		)
-		(property "LCSC" "C60490"
+		(property "LCSC" "C25744"
 			(at 69.85 156.21 0)
 			(hide yes)
